File: KiCad PCB Schematic files/SDR_Schematic_and_PCB_files/SDRReciever02.sch (KiCad schematic (older format))
At the start: 62 parts, among them J1 Conn_Coaxial, J10 I_0, J11 I_180, J12 Q_90, J13 Q_270, J16 5V, J17 4.3V, J2 AudioJack3, J3 FIL_I, J4 FIL_O, J5 CLK_1, J6 CLK_2, J7 CLK_0, Q1 PN2222A, Q2 BSS138, Q3 BSS138, U1 Si5351A-B-GT, U2 LM4562, U3 SN74CBT3253, Y1 ATS250

Commit message: Updated KiCad Schematic 1. Exchanged instrumentation amplifiers and following op amp low pass filters for a single set of low noise op amps with multiple feedback and two poles of attenuation. 2. Removed the buffer amp and voltage divider previously creating analog ground at the end of the voltage smoother since it is no longer needed. 3. Updated footprints and exchanged most through hole components for surface mount components 4. Updated crystal oscillator chip 5. Fixed counting order at output from tayloe mixer and input to amplifiers
Parts:
- C1, C3: footprint Capacitor_THT:C_Disc_D4.7mm_W2.5mm_P5.00mm -> Capacitor_SMD:C_0805_2012Metric
- C10, C11, C12, C13, C4: footprint Capacitor_THT:C_Disc_D5.1mm_W3.2mm_P5.00mm -> Capacitor_SMD:C_0805_2012Metric
- C14, C15, C16, C2, C5, C6, C7: footprint Capacitor_THT:C_Disc_D5.0mm_W2.5mm_P2.50mm -> Capacitor_SMD:C_0805_2012Metric
- C9: footprint Capacitor_THT:CP_Radial_D5.0mm_P2.00mm -> Capacitor_SMD:C_0805_2012Metric
- J3: value FIL_I -> FIL_IN
- J4: value FIL_O -> FIL_OUT
- L1: footprint Inductor_THT:L_Toroid_Vertical_L13.0mm_W6.5mm_P5.60mm -> Inductor_THT:L_Toroid_Vertical_L10.0mm_W5.0mm_P5.08mm
- L2: footprint Inductor_THT:L_Toroid_Vertical_L10.0mm_W5.0mm_P5.08mm -> Inductor_THT:L_Toroid_Vertical_L13.0mm_W6.5mm_P5.60mm
- R1, R10, R11, R12, R13, R14, R18, R19, R3, R4, R5: footprint Resistor_THT:R_Axial_DIN0207_L6.3mm_D2.5mm_P7.62mm_Horizontal -> Resistor_SMD:R_0805_2012Metric
- R7, R8: footprint (none) -> Resistor_SMD:R_0805_2012Metric
- Y1: value ATS250 -> CX3225SB; footprint Crystal:Crystal_HC49-U_Vertical -> Crystal:Crystal_SMD_Abracon_ABM8G-4Pin_3.2x2.5mm; symbol SDRReciever-rescue:Crystal-Device -> Device:Crystal_GND24; DigiKey (none) -> https://www.digikey.com/en/products/detail/kyocera-internat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
Connections:
- net GND: now also Y1.2, Y1.4
- net at U1.3 (XB): now also Y1.3; no longer Y1.2
Other:
- note added: "CX3225SB\n25 MHz crystal"
- note added: "Full Scale Input \nSignal Level Typ: 1.0 Vrms\nInput R = 55kΩ?????"
- note added: "Optional\nbypass jumper"
- note added: "T37-6 Toroid:\n11.9 turns"
- note added: "T50-6 Toroid: \n14.3 turns"
- note removed: "Full Scale Input \nSignal Level Typ: 1.0 Vrms\nInput R = 55kΩ."
- note removed: "NOTE:\nDouble check values of C5-C8\n100nf?"
- note removed: "T37-6 Toroid:\n-- turns"
- note removed: "T50-6 Toroid: \n-- turns"
- note removed: "The ATS250 is \na low-cost 25 \nMHz crystal\n\nCX3225\n25 MHz crystal"

Commit message: Removed diodes, added test point
Parts:
- removed D1, D2: 1N914, Diode_THT:D_DO-35_SOD27_P7.62mm_Horizontal, symbol SDRReciever-rescue:1N914-Diode
- added J8: 3.3V, Connector_PinHeader_2.54mm:PinHeader_1x01_P2.54mm_Vertical, symbol SDRReciever-rescue:Conn_01x01-Connector_Generic
Connections:
- net +3V3: now also J8.1 (Pin_1)
- net SCL_3V: no longer R21.2
Other:
- note removed: "Note:\nCheck all footprints\nExchange some through hole components for surface mount"
- note removed: "Voltage Protection Diodes:\nThese will prevent too large of signals \nfrom coming through"
- moved on the sheet: Q3
Changed lines of the file:
@@
 $EndComp
-Wire Wire Line
-	2750 2200 2750 2400
 Wire Wire Line
 	4250 2200 4250 2400
@@
 $EndComp
 $Comp
-L SDRReciever-rescue:1N914-Diode D2
-U 1 1 5EA1DE64
-P 2750 2050
-F 0 "D2" V 2796 1971 50  0000 R CNN
-F 1 "1N914" V 2705 1971 50  0000 R CNN
-F 2 "Diode_THT:D_DO-35_SOD27_P7.62mm_Horizontal" H 2750 1875 50  0001 C CNN
-F 3 "http://www.vishay.com/docs/85622/1n914.pdf" H 2750 2050 50  0001 C CNN
-	1    2750 2050
-	0    -1   -1   0
-$EndComp
-$Comp
 L Device:Crystal_GND24 Y1
 U 1 1 5EA4F383
@@
 	8050 2600 7850 2600
 Connection ~ 2000 2400
-Wire Wire Line
-	2000 2400 2350 2400
 $Comp
 L SDRReciever-rescue:Conn_01x01-Connector_Generic J3
@@
 $EndComp
 Connection ~ 2350 1900
-$Comp
-L SDRReciever-rescue:1N914-Diode D1
-U 1 1 5EA1C428
-P 2350 2050
-F 0 "D1" V 2304 2129 50  0000 L CNN
-F 1 "1N914" V 2395 2129 50  0000 L CNN
-F 2 "Diode_THT:D_DO-35_SOD27_P7.62mm_Horizontal" H 2350 1875 50  0001 C CNN
-F 3 "http://www.vishay.com/docs/85622/1n914.pdf" H 2350 2050 50  0001 C CNN
-	1    2350 2050
-	0    1    1    0
-$EndComp
 Wire Wire Line
 	2200 1900 2350 1900
-Wire Wire Line
-	2350 2200 2350 2400
 Wire Wire Line
 	2000 2350 2000 2400
@@
 Text Notes 2250 1325 0    50   ~ 0
 6-16MHz (3rd Order, Series-First Butterworth)\nBy doing Series-First, DC signals cannot pass through the capacitor (C2), \nallowing better control over the DC offset going into the op-amps
-Text Notes 2275 2675 0    50   ~ 0
-Voltage Protection Diodes:\nThese will prevent too large of signals \nfrom coming through
 Text Notes 8875 2100 0    50   ~ 0
 00 = 0°
@@
 Wire Notes Line
 	1800 650  650  650
-Connection ~ 2350 2400
 Wire Wire Line
 	4050 2400 4250 2400
-Wire Wire Line
-	2750 1900 3150 1900
-Wire Wire Line
-	2750 2400 4050 2400
-Wire Wire Line
-	2350 2400 2750 2400
-Wire Wire Line
-	2350 1900 2750 1900
 Wire Wire Line
 	7250 4425 6775 4425
@@
 Text Notes 1375 1650 0    50   ~ 0
 Antenna Connector
-Connection ~ 2750 2400
-Connection ~ 2750 1900
 Connection ~ 4050 2400
 Text Notes 2325 1600 0    50   ~ 0
@@
 Wire Wire Line
 	4450 6825 4450 6875
-Wire Wire Line
-	2400 6825 2800 6825
 Connection ~ 2400 6825
 Wire Wire Line
@@
 	4050 6825 4450 6825
 Connection ~ 4450 6825
-$Comp
-L Device:Q_NMOS_GSD Q3
-U 1 1 608C951F
-P 3750 8025
-F 0 "Q3" V 3999 8025 50  0000 C CNN
-F 1 "BSS138" V 4090 8025 50  0000 C CNN
-F 2 "Package_TO_SOT_SMD:SOT-23" H 3950 8125 50  0001 C CNN
-F 3 "~" H 3750 8025 50  0001 C CNN
-	1    3750 8025
-	0    1    1    0
-$EndComp
-Wire Wire Line
-	3550 8125 2800 8125
 $Comp
 L Device:Q_NMOS_GSD Q2
@@
 Wire Wire Line
 	3200 6825 3750 6825
-Wire Wire Line
-	3750 6825 3750 7825
 Connection ~ 3200 6825
 Wire Wire Line
@@
 Wire Wire Line
 	4050 7425 3400 7425
-Wire Wire Line
-	4450 8125 3950 8125
 Wire Wire Line
 	4450 7175 4450 7775
@@
 	2800 6825 3200 6825
 Wire Wire Line
-	2800 7175 2800 8125
-Connection ~ 2800 8125
-Wire Wire Line
-	2800 8125 2100 8125
-Wire Wire Line
 	4450 6675 4450 6825
 Wire Wire Line
 	4450 7775 4750 7775
-Connection ~ 4450 7775
-Wire Wire Line
-	4450 7775 4450 8125
 Text Label 4750 7775 0    50   ~ 0
 SCL_5V
@@
 Text Label 2100 7425 2    50   ~ 0
 SDA_3V
-Text Label 2100 8125 2    50   ~ 0
-SCL_3V
 Wire Wire Line
 	2400 7425 2100 7425
@@
 Q_LO
 Wire Wire Line
-	2400 6650 2400 6825
-Wire Wire Line
 	4050 7425 4150 7425
 Connection ~ 4050 7425
-Text Notes 6550 6825 0    50   ~ 0
-Note:\nCheck all footprints\nExchange some through hole components for surface mount
 $Comp
 L Amplifier_Operational:LM4562 U2
@@
 Text Notes 1700 4900 0    50   ~ 0
 Optional\nbypass jumper
+Wire Wire Line
+	2350 1900 3150 1900
+Wire Wire Line
+	2000 2400 4050 2400
+$Comp
+L SDRReciever-rescue:Conn_01x01-Connector_Generic J8
+U 1 1 60888163
+P 2200 6700
+F 0 "J8" H 2325 6750 50  0000 L CNN
+F 1 "3.3V" H 2300 6675 50  0000 L CNN
+F 2 "Connector_PinHeader_2.54mm:PinHeader_1x01_P2.54mm_Vertical" H 2200 6700 50  0001 C CNN
+F 3 "~" H 2200 6700 50  0001 C CNN
+	1    2200 6700
+	-1   0    0    1
+$EndComp
+Connection ~ 4450 7775
+Wire Wire Line
+	2400 6825 2800 6825
+Text Label 2100 7775 2    50   ~ 0
+SCL_3V
+Wire Wire Line
+	4450 7775 3950 7775
+$Comp
+L Device:Q_NMOS_GSD Q3
+U 1 1 608C951F
+P 3750 7675
+F 0 "Q3" V 3999 7675 50  0000 C CNN
+F 1 "BSS138" V 4090 7675 50  0000 C CNN
+F 2 "Package_TO_SOT_SMD:SOT-23" H 3950 7775 50  0001 C CNN
+F 3 "~" H 3750 7675 50  0001 C CNN
+	1    3750 7675
+	0    1    1    0
+$EndComp
+Wire Wire Line
+	2100 7775 3550 7775
+Wire Wire Line
+	3750 6825 3750 7475
+Wire Wire Line
+	2400 6650 2400 6700
+Connection ~ 2400 6700
+Wire Wire Line
+	2400 6700 2400 6825
 $EndSCHEMATC
