File: KiCad PCB Schematic files/SDR_Schematic_and_PCB_files/SDRReciever.kicad_pcb (KiCad board)
At the start: 2 copper layers, 100 x 100 mm, 78 parts, among them J1 Conn_Coaxial, J10 I_0, J11 I_180, J12 Q_90, J13 Q_270, J14 I_OUT, J15 Q_OUT, J16 5V, J17 4.3V, J18 Conn_01x02_Female, J19 Conn_01x02_Female, J2 AudioJack3, J3 FIL_I, J4 FIL_O, J5 CLK_2, J6 CLK_3, J7 CLK_1, J8 I_LO, J9 Q_LO, Q1 PN2222A, U1 Si5351A-B-GT, U2 74AC74, U3 SN74CBT3253, U4 INA821ID, U5 INA821ID, U6 OP213FPZ, Y1 Crystal

Commit message: Revision 0.3 of schematic Added bypass cap Added DC blocking caps Removed redudant resitors Added custom footprints Updated BNC connector footprint Updated audo jack footprint, schematic symbol, connections, and 3D model Updated comments Removed old PCB Created new blank PCB
Parts:
- removed A1: Arduino_Nano_v3.x, Module:Arduino_Nano
- removed C1, C3: 220pF, Capacitor_THT:C_Disc_D4.7mm_W2.5mm_P5.00mm
- removed C10, C11, C12, C13, C14, C17, C18, C23, C24, C4: 0.1u, Capacitor_THT:C_Disc_D5.1mm_W3.2mm_P5.00mm
- removed C15, C16, C9: 10uF, Capacitor_THT:CP_Radial_D5.0mm_P2.00mm
- removed C19, C20: 220p, Capacitor_THT:C_Disc_D4.7mm_W2.5mm_P5.00mm
- removed C2: 1nF, Capacitor_THT:C_Disc_D5.0mm_W2.5mm_P2.50mm
- removed C21, C22, C5, C6, C7, C8: 100p, Capacitor_THT:C_Disc_D5.0mm_W2.5mm_P2.50mm
- removed D1, D2: 1N914, Diode_THT:D_DO-35_SOD27_P7.62mm_Horizontal
- removed J1: Conn_Coaxial, Connector_Coaxial:SMA_Molex_73251-1153_EdgeMount_Horizontal
- removed J10: I_0, Connector_PinHeader_2.54mm:PinHeader_1x01_P2.54mm_Vertical
- removed J11: I_180, Connector_PinHeader_2.54mm:PinHeader_1x01_P2.54mm_Vertical
- removed J12: Q_90, Connector_PinHeader_2.54mm:PinHeader_1x01_P2.54mm_Vertical
- removed J13: Q_270, Connector_PinHeader_2.54mm:PinHeader_1x01_P2.54mm_Vertical
- removed J14: I_OUT, Connector_PinHeader_2.54mm:PinHeader_1x01_P2.54mm_Vertical
- removed J15: Q_OUT, Connector_PinHeader_2.54mm:PinHeader_1x01_P2.54mm_Vertical
- removed J16: 5V, Connector_PinHeader_2.54mm:PinHeader_1x01_P2.54mm_Vertical
- removed J17: 4.3V, Connector_PinHeader_2.54mm:PinHeader_1x01_P2.54mm_Vertical
- removed J18, J19: Conn_01x02_Female, Connector_PinSocket_2.54mm:PinSocket_1x02_P2.54mm_Vertical
- removed J2: AudioJack3, Connector_Audio:Jack_3.5mm_Switronic_ST-005-G_horizontal
- removed J3: FIL_I, Connector_PinHeader_2.54mm:PinHeader_1x01_P2.54mm_Vertical
- removed J4: FIL_O, Connector_PinHeader_2.54mm:PinHeader_1x01_P2.54mm_Vertical
- removed J5: CLK_2, Connector_PinHeader_2.54mm:PinHeader_1x01_P2.54mm_Vertical
- removed J6: CLK_3, Connector_PinHeader_2.54mm:PinHeader_1x01_P2.54mm_Vertical
- removed J7: CLK_1, Connector_PinHeader_2.54mm:PinHeader_1x01_P2.54mm_Vertical
- removed J8: I_LO, Connector_PinHeader_2.54mm:PinHeader_1x01_P2.54mm_Vertical
- removed J9: Q_LO, Connector_PinHeader_2.54mm:PinHeader_1x01_P2.54mm_Vertical
- removed JP1, JP2, JP3, JP4: Jumper_NC_Small, Connector_PinHeader_2.54mm:PinHeader_1x02_P2.54mm_Vertical
- removed L1, L3: 1.3uH, Inductor_THT:L_Toroid_Vertical_L13.0mm_W6.5mm_P5.60mm
- removed L2: 200nH, Inductor_THT:L_Toroid_Vertical_L10.0mm_W5.0mm_P5.08mm
- removed Q1: PN2222A, Package_TO_SOT_THT:TO-92_Inline
- removed R1: 1k, Resistor_THT:R_Axial_DIN0207_L6.3mm_D2.5mm_P7.62mm_Horizontal
- removed R10, R11, R12, R5: 50, Resistor_THT:R_Axial_DIN0207_L6.3mm_D2.5mm_P7.62mm_Horizontal
- removed R13, R14: 8.2k, Resistor_THT:R_Axial_DIN0207_L6.3mm_D2.5mm_P7.62mm_Horizontal
- removed R15, R16: 15k, Resistor_THT:R_Axial_DIN0207_L6.3mm_D2.5mm_P7.62mm_Horizontal
- removed R17, R2, R7, R8: 10k, Resistor_THT:R_Axial_DIN0207_L6.3mm_D2.5mm_P7.62mm_Horizontal
- removed R3, R4: 33, Resistor_THT:R_Axial_DIN0207_L6.3mm_D2.5mm_P7.62mm_Horizontal
- removed R6, R9: 100, Resistor_THT:R_Axial_DIN0207_L6.3mm_D2.5mm_P7.62mm_Horizontal
- removed U1: Si5351A-B-GT, Package_SO:MSOP-10_3x3mm_P0.5mm
- removed U2: 74AC74, Package_DIP:DIP-14_W7.62mm
- removed U3: SN74CBT3253, Package_SO:SOIC-16_3.9x9.9mm_P1.27mm
- removed U4, U5: INA821ID, import_footprint:SOIC127P600X175-8N
- removed U6: OP213FPZ, Imported_Footprints:OP213FPZ
- removed Y1: Crystal, Crystal:Crystal_HC49-U_Vertical
Routing:
- net +4.3V: track 215.4 -> 0.00 mm
- net +3V3: track 92.6 -> 0.00 mm
- net /Q_LO: track 85.6 -> 0.00 mm, vias 1 -> 0
- net /I_LO: track 76.3 -> 0.00 mm, vias 1 -> 0
- net /FIL_OUT: track 72.8 -> 0.00 mm
- net GNDA: track 71.2 -> 0.00 mm, vias 1 -> 0
- net +5V: track 65.1 -> 0.00 mm
- net Net-(J15-Pad1): track 42.2 -> 0.00 mm, vias 1 -> 0
- net Net-(R10-Pad2): track 38.5 -> 0.00 mm, vias 1 -> 0
- net Net-(C2-Pad1): track 37.0 -> 0.00 mm
- net Net-(J7-Pad1): track 33.4 -> 0.00 mm
- net Net-(R5-Pad2): track 30.6 -> 0.00 mm
- net Net-(J1-Pad2): track 29.5 -> 0.00 mm
- net Net-(A1-Pad29): track 29.2 -> 0.00 mm
- net Net-(J14-Pad1): track 27.5 -> 0.00 mm, vias 2 -> 0
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- removed copper zone on B.Cu, net GND
- removed copper zone on F.Cu, net GND
Other:
- board outline removed
- rule pad_to_mask_clearance: 0.051 -> 0
- board text removed: "0.1uF"
- board text removed: "2.15V Analog Ground Bias"
- board text removed: "2.15V Bias"
- board text removed: "25MHz Crystal"
- board text removed: "2nd Order Low Pass Filter"
- board text removed: "4:1 DeMux Tayloe Mixer"
- board text removed: "74AC74 Dual D Flip Flops"
- board text removed: "CLK_1 (LO)"
- board text removed: "CLK_2"
- board text removed: "CLK_3"
- board text removed: "Dual Low-Noise Single Supply Op Amp"
- board text removed: "Gain Resistor"
- board text removed: "Johnson Counter CLK/4 Circuit"
- board text removed: "Konrad McClure Caleb Froelich ENGR 357 - Electronics II"
- board text removed: "LC Bandpass Filter 5-18MHz"
- board text removed: "Low Cost SDR Receiver"
- board text removed: "Low Noise Intrstumentation Amplifiers"
- board text removed: "Rev: 2"
- board text removed: "Test Gain Resistors"
- board text removed: "Voltage Smoother"
